File: pcb/custom_keyboard.kicad_pcb (KiCad board)
At the start: 2 copper layers, 385.9 x 133.7 mm, 175 parts, among them SW1 SW_Push, SW10 SW_Push, SW11 SW_Push, SW12 SW_Push, SW13 SW_Push, SW14 SW_Push, SW15 SW_Push, SW16 SW_Push, SW17 SW_Push, SW18 SW_Push, SW19 SW_Push, SW2 SW_Push, SW20 SW_Push, SW21 SW_Push, SW22 SW_Push, SW23 SW_Push, SW24 SW_Push, SW25 SW_Push, SW26 SW_Push, SW27 SW_Push, SW28 SW_Push, SW29 SW_Push, SW3 SW_Push, SW30 SW_Push, SW31 SW_Push, SW32 SW_Push, SW33 SW_Push, SW34 SW_Push, SW35 SW_Push, SW36 SW_Push, SW37 SW_Push, SW38 SW_Push, SW39 SW_Push, SW4 SW_Push, SW40 SW_Push, SW41 SW_Push, SW42 SW_Push, SW43 SW_Push, SW44 SW_Push, SW45 SW_Push, SW46 SW_Push, SW47 SW_Push, SW48 SW_Push, SW49 SW_Push, SW5 SW_Push, SW50 SW_Push, SW51 SW_Push, SW52 SW_Push, SW53 SW_Push, SW54 SW_Push, SW55 SW_Push, SW56 SW_Push, SW57 SW_Push, SW58 SW_Push, SW59 SW_Push, SW6 SW_Push, SW60 SW_Push, SW61 SW_Push, SW62 SW_Push, SW63 SW_Push, SW64 SW_Push, SW65 SW_Push, SW66 SW_Push, SW67 SW_Push, SW68 SW_Push, SW69 SW_Push, SW7 SW_Push, SW70 SW_Push, SW71 SW_Push, SW72 SW_Push, SW73 SW_Push, SW74 SW_Push, SW75 SW_Push, SW76 SW_Push, SW77 SW_Push, SW78 SW_Push, SW79 SW_Push, SW8 SW_Push, SW80 SW_Push, SW81 SW_Push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

Commit message: Add progress from today
Parts:
- SW34: footprint PCM_marbastlib-mx:SW_MX_1u -> PCM_marbastlib-mx:SW_MX_1.5u
- SW48: footprint PCM_marbastlib-mx:SW_MX_1u -> PCM_marbastlib-mx:SW_MX_1.75u
- SW61, SW75, SW76, SW77, SW79, SW80, SW81, SW82: footprint PCM_marbastlib-mx:SW_MX_1u -> PCM_marbastlib-mx:SW_MX_1.25u
- moved SW14 28.6 mm to (133.3, 31.3)
- moved SW15 28.6 mm to (152.4, 31.3)
- moved SW16 28.6 mm to (171.4, 31.3)
- moved D16 28.5 mm to (181.0, 36.0)
- moved D14 28.5 mm to (142.9, 36.0)
- moved D15 28.5 mm to (161.9, 36.0)
- moved D32 19.2 mm to (161.9, 55.2)
- moved D31 19.0 mm to (142.9, 55.1)
- moved D33 19.0 mm to (181.0, 55.1)
- moved SW31 19.0 mm to (133.3, 50.3)
- moved SW32 19.0 mm to (152.4, 50.3)
- moved SW33 19.0 mm to (171.4, 50.3)
Routing:
- net /KBC13: track 353.9 -> 324.1 mm
- net /KBC15: track 311.8 -> 330.8 mm
- net /KBC14: track 404.4 -> 423.5 mm
- net /KBR3: track 415.6 -> 433.7 mm
- net /KBR4: track 465.5 -> 480.9 mm

Commit message: Add mounting holes and custom components
Parts:
- added D14: 1N4148, Diode_THT:D_DO-35_SOD27_P7.62mm_Horizontal, F.Cu at (359.5, 6.83)
- added D76: 1N4148, Diode_THT:D_DO-35_SOD27_P7.62mm_Horizontal, F.Cu at (85.9, 109.5)
- added REF**: MountingHole_3mm, MountingHole:MountingHole_3mm, F.Cu at (156.0, 114.3)
- added REF**: MountingHole_3mm, MountingHole:MountingHole_3mm, F.Cu at (-9.53, 75.0)
- added REF**: MountingHole_3mm, MountingHole:MountingHole_3mm, F.Cu at (110.7, 114.3)
- added REF**: MountingHole_3mm, MountingHole:MountingHole_3mm, F.Cu at (283.4, 114.3)
- added REF**: MountingHole_3mm, MountingHole:MountingHole_3mm, F.Cu at (367.9, 14.3)
- added REF**: MountingHole_3mm, MountingHole:MountingHole_3mm, F.Cu at (109.5, -9.53)
- added REF**: MountingHole_3mm, MountingHole:MountingHole_3mm, F.Cu at (-9.53, 47.6)
- added REF**: MountingHole_3mm, MountingHole:MountingHole_3mm, F.Cu at (-8.33, 113.1)
- added REF**: MountingHole_3mm, MountingHole:MountingHole_3mm, F.Cu at (303.6, 114.3)
- added REF**: MountingHole_3mm, MountingHole:MountingHole_3mm, F.Cu at (366.7, 83.3)
- added REF**: MountingHole_3mm, MountingHole:MountingHole_3mm, F.Cu at (195.3, -9.53)
- added REF**: MountingHole_3mm, MountingHole:MountingHole_3mm, F.Cu at (-9.53, -9.53)
- added SW1: RotaryEncoder_Switch, Rotary_Encoder:RotaryEncoder_Alps_EC11E-Switch_Vertical_H20mm, F.Cu at (352.5, -6.98)
- added SW76: SW_Push, PCM_marbastlib-mx:SW_MX_1.25u, F.Cu at (73.8, 104.8)
- added U1: ER_OLEDM0.91_1x-I2C, Display:ER_OLEDM0.91_1x-I2C, F.Cu at (311.9, -0.67)
- A1: footprint Module:RaspberryPi_Pico_Common_SMD -> Module:RaspberryPi_Pico_SMD
- S4: footprint PCM_marbastlib-mx:STAB_MX_6.25u -> PCM_marbastlib-mx:STAB_MX_5u
- moved S4 198.0 mm to (133.5, 104.8)
- moved SW87 198.0 mm to (133.5, 105.1)
- moved SW14 185.9 mm to (266.7, 0.01)
- moved SW31 185.9 mm to (357.4, 28.6)
- moved SW47 185.9 mm to (357.4, 47.6)
- moved SW86 185.9 mm to (357.4, 104.8)
- moved D1 185.9 mm to (9.53, 4.77)
- moved D10 185.9 mm to (219.1, 4.77)
- moved D11 185.9 mm to (238.1, 4.77)
- moved D17 185.9 mm to (366.9, 33.3)
- moved D18 185.9 mm to (9.53, 33.3)
- moved D19 185.9 mm to (28.6, 33.3)
- moved D2 185.9 mm to (47.6, 4.77)
- moved D20 185.9 mm to (47.6, 33.3)
- moved D21 185.9 mm to (66.7, 33.3)
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- renumbered D14 to D15, D15 to D16, D16 to D17, D17 to D18, D18 to D19, D19 to D20, D20 to D21, D21 to D22, D22 to D23, D23 to D24, D24 to D25, D25 to D26, D26 to D27, D27 to D28, D28 to D29, D29 to D30, D30 to D31, D34 to D32, D35 to D33, D36 to D34, D37 to D35, D38 to D36, D39 to D37, D40 to D38, D41 to D39, D42 to D40, D43 to D41, D44 to D42, D45 to D43, D46 to D44, D47 to D45, D31 to D46, D33 to D47, D32 to D48, D48 to D49, D49 to D50, D50 to D51, D51 to D52, D52 to D53, D53 to D54, D54 to D55, D55 to D56, D56 to D57, D57 to D58, D58 to D59, D59 to D60, D60 to D61, D61 to D62, D62 to D63, D63 to D64, D64 to D65, D65 to D66, D66 to D67, D67 to D68, D68 to D69, D69 to D70, D70 to D71, D71 to D72, D72 to D73, D73 to D74, D74 to D75, D75 to D77, D76 to D78, D77 to D79, D78 to D80, D79 to D81, D80 to D82, D81 to D83, D82 to D84, D83 to D85, D84 to D86, D85 to D87, SW9 to SW10, SW10 to SW11, SW11 to SW12, SW12 to SW13, SW13 to SW14, SW17 to SW15, SW18 to SW16, SW19 to SW17, SW20 to SW18, SW21 to SW19, SW1 to SW2, SW22 to SW20, SW23 to SW21, SW24 to SW22, SW25 to SW23, SW26 to SW24, SW27 to SW25, SW28 to SW26, SW29 to SW27, SW30 to SW28, SW14 to SW29, SW2 to SW3, SW15 to SW30, SW16 to SW31, SW34 to SW32, SW35 to SW33, SW36 to SW34, SW37 to SW35, SW38 to SW36, SW39 to SW37, SW40 to SW38, SW41 to SW39, SW3 to SW4, SW42 to SW40, SW43 to SW41, SW44 to SW42, SW45 to SW43, SW46 to SW44, SW31 to SW45, SW32 to SW46, SW33 to SW47, SW47 to SW48, SW48 to SW49, SW4 to SW5, SW49 to SW50, SW50 to SW51, SW51 to SW52, SW52 to SW53, SW53 to SW54, SW54 to SW55, SW55 to SW56, SW56 to SW57, SW57 to SW58, SW58 to SW59, SW5 to SW6, SW59 to SW60, SW60 to SW61, SW61 to SW62, SW62 to SW63, SW63 to SW64, SW64 to SW65, SW65 to SW66, SW66 to SW67, SW67 to SW68, SW68 to SW69, SW6 to SW7, SW69 to SW70, SW70 to SW71, SW71 to SW72, SW72 to SW73, SW73 to SW74, SW74 to SW75, SW75 to SW77, SW76 to SW78, SW77 to SW79, SW7 to SW8, SW79 to SW80, SW80 to SW81, SW81 to SW82, SW82 to SW83, SW83 to SW84, SW84 to SW85, SW85 to SW86, SW78 to SW87, SW8 to SW9
Connections:
- A1 pad 29: unconnected-(A1-GPIO22-Pad29) -> /GPIO22
- A1 pad 31: unconnected-(A1-GPIO26_ADC0-Pad31) -> /GPIO26
- A1 pad 32: unconnected-(A1-GPIO27_ADC1-Pad32) -> /GPIO27
- A1 pad 34: unconnected-(A1-GPIO28_ADC2-Pad34) -> /GPIO28
- A1 pad 36: unconnected-(A1-3V3-Pad36) -> /3V3
Routing:
- net /KBR5: track 371.7 -> 457.9 mm, vias 0 -> 2
- net /KBC10: track 258.6 -> 332.3 mm, vias 3 -> 4
- net /KBC15: track 330.8 -> 262.2 mm, vias 5 -> 4
- net /GPIO27: track 0.00 -> 64.9 mm, vias 0 -> 2
- net /GPIO28: track 0.00 -> 51.7 mm, vias 0 -> 2
- net /GPIO26: track 0.00 -> 36.5 mm, vias 0 -> 1
- net /GPIO22: track 0.00 -> 26.9 mm, vias 0 -> 1
- net /KBC3: track 328.2 -> 352.2 mm
- net /KBC5: track 293.3 -> 279.0 mm
- net Net-(D80-A): track 57.9 -> 45.7 mm
- net Net-(D76-A): track 0.00 -> 10.4 mm
- net /3V3: track 0.00 -> 9.47 mm
- net Net-(D14-A): track 0.00 -> 8.87 mm
- net /GND: track 0.00 -> 5.95 mm, vias 0 -> 13
- net /KBC7: track 301.0 -> 296.6 mm
